File: sumorobot-shield-pcb.brd (EAGLE design)
At the start: 58.6 x 53.3 mm, 29 parts

Commit message: updated schematics and board + renaming
Parts:
- removed U$2: (no value), arduino_uno:ROBOKODING-LOGO
- removed U$3: (no value), arduino_uno:OPENSOURCE-LOGO
- added LOGO1: ROBOKODING-LOGOL, robokoding-logo:ROBOKODING-LOGO-L
- added LOGO2: OSHW-LOGOL, SparkFun-Aesthetics:OSHW-LOGO-L
Other:
- board text added: "Sumoshield V0.1"
- board text removed: "SUMOINO V3.0"
Changed lines of the file:
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@@
 <?xml version="1.0" encoding="utf-8"?>
 <!DOCTYPE eagle SYSTEM "eagle.dtd">
-<eagle version="6.5.0">
+<eagle version="7.1.0">
 <drawing>
 <settings>
@@
 <setting verticaltext="up"/>
 </settings>
-<grid distance="0.1" unitdist="mm" unit="mm" style="lines" multiple="1" display="yes" altdistance="0.1" altunitdist="mm" altunit="mm"/>
+<grid distance="0.5" unitdist="mm" unit="mm" style="lines" multiple="1" display="yes" altdistance="0.5" altunitdist="mm" altunit="mm"/>
 <layers>
 <layer number="1" name="Top" color="4" fill="1" visible="yes" active="yes"/>
@@
 <layer number="54" name="bGND_GNDA" color="1" fill="9" visible="no" active="no"/>
 <layer number="56" name="wert" color="7" fill="1" visible="no" active="yes"/>
+<layer number="57" name="tCAD" color="7" fill="1" visible="no" active="no"/>
 <layer number="91" name="Nets" color="2" fill="1" visible="no" active="no"/>
 <layer number="92" name="Busses" color="1" fill="1" visible="no" active="no"/>
@@
 <layer number="97" name="Info" color="7" fill="1" visible="no" active="no"/>
 <layer number="98" name="Guide" color="6" fill="1" visible="no" active="no"/>
+<layer number="99" name="SpiceOrder" color="7" fill="1" visible="no" active="no"/>
 <layer number="100" name="Muster" color="7" fill="1" visible="no" active="no"/>
 <layer number="101" name="Patch_Top" color="12" fill="4" visible="no" active="yes"/>
@@
 <layer number="110" name="fp0" color="7" fill="1" visible="no" active="yes"/>
 <layer number="111" name="border" color="15" fill="1" visible="no" active="yes"/>
+<layer number="112" name="tSilk" color="7" fill="1" visible="yes" active="yes"/>
+<layer number="113" name="IDFDebug" color="4" fill="1" visible="yes" active="yes"/>
 <layer number="116" name="Patch_BOT" color="9" fill="4" visible="no" active="yes"/>
 <layer number="121" name="_tsilk" color="7" fill="1" visible="no" active="yes"/>
@@
 <layer number="125" name="_tNames" color="7" fill="1" visible="no" active="yes"/>
 <layer number="126" name="_bNames" color="7" fill="1" visible="no" active="yes"/>
+<layer number="127" name="_tValues" color="7" fill="1" visible="yes" active="yes"/>
+<layer number="128" name="_bValues" color="7" fill="1" visible="yes" active="yes"/>
 <layer number="131" name="tAdjust" color="7" fill="1" visible="no" active="yes"/>
 <layer number="132" name="bAdjust" color="7" fill="1" visible="no" active="yes"/>
 <layer number="144" name="Drill_legend" color="7" fill="1" visible="no" active="yes"/>
+<layer number="150" name="Notes" color="7" fill="1" visible="yes" active="yes"/>
 <layer number="151" name="HeatSink" color="7" fill="1" visible="no" active="yes"/>
+<layer number="152" name="_bDocu" color="7" fill="1" visible="yes" active="yes"/>
+<layer number="153" name="FabDoc1" color="7" fill="1" visible="yes" active="yes"/>
+<layer number="154" name="FabDoc2" color="7" fill="1" visible="yes" active="yes"/>
+<layer number="155" name="FabDoc3" color="7" fill="1" visible="yes" active="yes"/>
 <layer number="199" name="Contour" color="7" fill="1" visible="no" active="yes"/>
 <layer number="200" name="200bmp" color="1" fill="10" visible="no" active="yes"/>
@@
 <layer number="223" name="223bmp" color="7" fill="1" visible="no" active="yes"/>
 <layer number="224" name="224bmp" color="7" fill="1" visible="no" active="yes"/>
+<layer number="248" name="Housing" color="7" fill="1" visible="yes" active="yes"/>
+<layer number="249" name="Edge" color="7" fill="1" visible="yes" active="yes"/>
 <layer number="250" name="Descript" color="7" fill="1" visible="no" active="no"/>
 <layer number="251" name="SMDround" color="7" fill="1" visible="no" active="no"/>
@@
 <wire x1="0" y1="11.5" x2="0" y2="0" width="0" layer="20"/>
 <wire x1="0" y1="53.34" x2="47.52" y2="53.34" width="0" layer="20"/>
-<text x="1.8" y="51.7" size="1.9304" layer="21" ratio="15" rot="SR270">SUMOINO V3.0</text>
+<text x="1.8" y="51.7" size="1.9304" layer="21" ratio="15" rot="SR270">Sumoshield V0.1</text>
 <text x="34.8" y="11.8" size="1.9304" layer="21" ratio="15" rot="R90">0</text>
 <text x="35.4" y="13.2" size="1.9304" layer="21" ratio="15" rot="SR270">1</text>
@@
 <pass name="Default">
 <param name="RoutingGrid" value="50mil"/>
+<param name="AutoGrid" value="1"/>
+<param name="Efforts" value="0"/>
+<param name="TopRouterVariant" value="1"/>
 <param name="tpViaShape" value="round"/>
 <param name="PrefDir.1" value="|"/>
@@
 <element name="S1" library="switch-misc" package="9077-2" value="" x="27.9" y="8.3" rot="R180"/>
 <element name="S2" library="switch-misc" package="9077-2" value="" x="28.1" y="24.9"/>
-<element name="U$2" library="arduino_uno" package="ROBOKODING-LOGO" value="" x="1.8" y="29.9" rot="R270"/>
-<element name="U$3" library="arduino_uno" package="OPENSOURCE-LOGO" value="" x="11.9" y="27.2" rot="R270"/>
+<element name="LOGO1" library="robokoding-logo" package="ROBOKODING-LOGO-L" value="ROBOKODING-LOGOL" x="1.85" y="30.1" rot="R270"/>
+<element name="LOGO2" library="SparkFun-Aesthetics" package="OSHW-LOGO-L" value="OSHW-LOGOL" x="16" y="22" rot="R270"/>
 </elements>
 <signals>
@@
 <signal name="GND">
 <contactref element="U$1" pad="GND"/>
-<contactref element="U$1" pad="GND1"/>
 <contactref element="LED1" pad="K"/>
-<contactref element="U$1" pad="GND2"/>
 <contactref element="C2" pad="-"/>
 <contactref element="LM2940T" pad="GND"/>
@@
 <contactref element="J8" pad="2"/>
 <contactref element="J1" pad="3"/>
-<contactref element="BLUETOOTH" pad="GND0"/>
 <contactref element="LED2" pad="K"/>
 <contactref element="J9" pad="2"/>
@@
 <contactref element="J7" pad="1"/>
 <contactref element="J7" pad="2"/>
-<contactref element="R1" pad="1"/>
 <contactref element="S3" pad="3"/>
 <contactref element="S3" pad="4"/>
@@
 <vertex x="52" y="54"/>
 </polygon>
+<contactref element="U$1" pad="GND1"/>
+<contactref element="U$1" pad="GND2"/>
+<contactref element="BLUETOOTH" pad="GND0"/>
+<contactref element="R1" pad="1"/>
 </signal>
 <signal name="N$14">

Commit message: updated sumorobot shield
Parts:
- C1: value 1000uF +5V -> 5V; device rcl:E2,5-7 -> rcl:E3,5-8
- C2: value 330uF +25V -> 25V
- LED1: value (none) -> BT STAT
- LED2: value (none) -> POWER
- moved C1 1.68 mm to (47.6, 18.2)
- moved LOGO2 0.70 mm to (15.3, 22.0)
- moved R3 0.15 mm to (49.4, 27.9), flipped to the top
Routing:
- net VCC: track 100.9 -> 102.5 mm
