File: sumorobot-shield-pcb.sch (EAGLE design)
At the start: 27 parts

Commit message: updated schematics and board + renaming
Parts:
- added LOGO1: ROBOKODING-LOGOL, robokoding-logo:ROBOKODING-LOGOL
- added LOGO2: OSHW-LOGOL, SparkFun-Aesthetics:OSHW-LOGOL
Other:
- moved on the sheet: C5, J1, J4, J5, J6, J7, LED1, R1, R2, R4, S2, S3

Commit message: updated sumorobot shield
Parts:
- C1: value 1000uF +5V -> 5V; device rcl:CPOL-EUE2.5-7 -> rcl:CPOL-EUE3.5-8
- C2: value 330uF +25V -> 25V
- LED1: value (none) -> BT STAT
- LED2: value (none) -> POWER
Changed lines of the file:
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@@
 <?xml version="1.0" encoding="utf-8"?>
 <!DOCTYPE eagle SYSTEM "eagle.dtd">
-<eagle version="7.1.0">
+<eagle version="6.5.0">
 <drawing>
 <settings>
@@
 <part name="U$1" library="arduino_uno" deviceset="SUMOINO-SHIELD" device="" value="SUMOINO-SHIELD"/>
 <part name="J10" library="con-lstb" deviceset="MA03-2" device=""/>
-<part name="C1" library="rcl" deviceset="CPOL-EU" device="E2.5-7" value="1000uF +5V"/>
-<part name="C2" library="rcl" deviceset="CPOL-EU" device="E2.5-7" value="330uF +25V"/>
+<part name="C1" library="rcl" deviceset="CPOL-EU" device="E3.5-8" value="5V"/>
+<part name="C2" library="rcl" deviceset="CPOL-EU" device="E2.5-7" value="25V"/>
 <part name="LM2940T" library="v-reg" deviceset="78XXL" device=""/>
 <part name="J9" library="con-lstb" deviceset="MA03-2" device=""/>
@@
 <part name="C5" library="rcl" deviceset="CPOL-EU" device="E5-4" value="0.1uF"/>
 <part name="J1" library="pinhead" deviceset="PINHD-1X3" device=""/>
-<part name="LED1" library="led" deviceset="LED" device="5MM"/>
+<part name="LED1" library="led" deviceset="LED" device="5MM" value="BT STAT"/>
 <part name="R2" library="rcl" deviceset="R-EU_" device="0204/7" value="300"/>
 <part name="GND6" library="supply1" deviceset="GND" device=""/>
@@
 <part name="GND16" library="supply1" deviceset="GND" device=""/>
 <part name="GND17" library="supply1" deviceset="GND" device=""/>
-<part name="LED2" library="led" deviceset="LED" device="5MM"/>
+<part name="LED2" library="led" deviceset="LED" device="5MM" value="POWER"/>
 <part name="R3" library="rcl" deviceset="R-EU_" device="0204/7" value="300"/>
 <part name="GND19" library="supply1" deviceset="GND" device=""/>
